File: pcb_design/EVKA_position_v4/EVKA_position_v4.kicad_pcb (KiCad board)
At the start: 2 copper layers, 110 x 80 mm, 43 parts, among them J1 THETA, J2 PHI, J3 WIRE, J4 Barrel_Jack_Switch, J5 LiPo 1S, J6 BENCH_5V, SW1 SW_DPDT_x2, U1 ESP32-S3-DEVKITC-1-N16R8V Upd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

Commit message: fix: remap v4 theta and wire ports
Parts:
- J1: value THETA -> WIRE
- J3: value WIRE -> THETA
Connections:
- J1 pad 1: /THETA_A_IN -> /WIRE_A_IN
- J1 pad 3: /THETA_B_IN -> /WIRE_B_IN
- J3 pad 1: /WIRE_A_IN -> /THETA_A_IN
- J3 pad 3: /WIRE_B_IN -> /THETA_B_IN
- R_TOP1 pad 2: /THETA_A_IN -> /WIRE_A_IN
- R_TOP2 pad 1: /THETA_B_IN -> /WIRE_B_IN
- R_TOP5 pad 2: /WIRE_A_IN -> /THETA_A_IN
- R_TOP6 pad 2: /WIRE_B_IN -> /THETA_B_IN
Changed lines of the file:
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@@
 			(layers "*.Cu" "*.Mask")
 			(remove_unused_layers no)
-			(net "/WIRE_B_IN")
+			(net "/THETA_B_IN")
 			(pintype "passive")
 		)
@@
 			)
 		)
-		(property "Value" "THETA"
+		(property "Value" "WIRE"
 			(at 14.986 -4.318 90)
 			(layer "F.Fab")
@@
 			(remove_unused_layers no)
 			(roundrect_rratio 0.096154)
-			(net "/THETA_A_IN")
+			(net "/WIRE_A_IN")
 			(pinfunction "Pin_1_1")
 			(pintype "passive")
@@
 			(layers "*.Cu" "*.Mask")
 			(remove_unused_layers no)
-			(net "/THETA_B_IN")
+			(net "/WIRE_B_IN")
 			(pinfunction "Pin_3_3")
 			(pintype "passive")
@@
 			(layers "*.Cu" "*.Mask")
 			(remove_unused_layers no)
-			(net "/THETA_A_IN")
+			(net "/WIRE_A_IN")
 			(pintype "passive")
 		)
@@
 			(layers "*.Cu" "*.Mask")
 			(remove_unused_layers no)
-			(net "/WIRE_A_IN")
+			(net "/THETA_A_IN")
 			(pintype "passive")
 		)
@@
 			)
 		)
-		(property "Value" "WIRE"
+		(property "Value" "THETA"
 			(at 15.494 -4.318 90)
 			(layer "F.Fab")
@@
 			(remove_unused_layers no)
 			(roundrect_rratio 0.096154)
-			(net "/WIRE_A_IN")
+			(net "/THETA_A_IN")
 			(pinfunction "Pin_1_1")
 			(pintype "passive")
@@
 			(layers "*.Cu" "*.Mask")
 			(remove_unused_layers no)
-			(net "/WIRE_B_IN")
+			(net "/THETA_B_IN")
 			(pinfunction "Pin_3_3")
 			(pintype "passive")
@@
 			(layers "*.Cu" "*.Mask")
 			(remove_unused_layers no)
-			(net "/THETA_B_IN")
+			(net "/WIRE_B_IN")
 			(pintype "passive")
 		)
@@
 		(width 1)
 		(layer "F.Cu")
-		(net "/WIRE_B_IN")
+		(net "/THETA_B_IN")
 	)
 	(segment
@@
 		(width 1)
 		(layer "F.Cu")
-		(net "/WIRE_B_IN")
+		(net "/THETA_B_IN")
 	)
 	(segment
@@
 		(width 1)
 		(layer "F.Cu")
-		(net "/WIRE_B_IN")
+		(net "/THETA_B_IN")
 	)
 	(segment
@@
 		(width 1)
 		(layer "F.Cu")
-		(net "/THETA_A_IN")
+		(net "/WIRE_A_IN")
 	)
 	(segment
@@
 		(width 1)
 		(layer "F.Cu")
-		(net "/THETA_A_IN")
+		(net "/WIRE_A_IN")
 	)
 	(segment
@@
 		(width 1)
 		(layer "F.Cu")
-		(net "/THETA_B_IN")
+		(net "/WIRE_B_IN")
 	)
 	(segment
@@
 		(width 1)
 		(layer "F.Cu")
-		(net "/THETA_B_IN")
+		(net "/WIRE_B_IN")
 	)
 	(segment
@@
 		(width 1)
 		(layer "F.Cu")
-		(net "/THETA_B_IN")
+		(net "/WIRE_B_IN")
 	)
 	(segment
@@
 		(width 1)
 		(layer "F.Cu")
-		(net "/WIRE_A_IN")
+		(net "/THETA_A_IN")
 	)
 	(segment
@@
 		(width 1)
 		(layer "F.Cu")
-		(net "/WIRE_A_IN")
+		(net "/THETA_A_IN")
 	)
 	(segment
