File: pcb_design/EVKA_position_v4/EVKA_position_v4.kicad_sch (KiCad schematic)
At the start: 43 parts, among them J1 THETA, J2 PHI, J3 WIRE, J4 Barrel_Jack_Switch, J5 LiPo 1S, J6 BENCH_5V, SW1 SW_DPDT_x2, U1 ESP32-S3-DEVKITC-1-N16R8V Upd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

Commit message: fix: remap v4 theta and wire ports
Parts:
- J1: value THETA -> WIRE
- J3: value WIRE -> THETA
Connections:
- net THETA_A_IN: now also J3.1 (Pin_1), R_TOP5.2; no longer J1.1 (Pin_1), R_TOP1.2
- net THETA_B_IN: now also J3.3 (Pin_3), R_TOP6.2; no longer J1.3 (Pin_3), R_TOP2.1
- net WIRE_A_IN: now also J1.1 (Pin_1), R_TOP1.2; no longer J3.1 (Pin_1), R_TOP5.2
- net WIRE_B_IN: now also J1.3 (Pin_3), R_TOP2.1; no longer J3.3 (Pin_3), R_TOP6.2
Changed lines of the file:
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@@
 		)
 	)
-	(label "WIRE_B_IN"
+	(label "THETA_B_IN"
 		(at 196.85 156.21 0)
 		(effects
@@
 		)
 	)
-	(label "THETA_B_IN"
+	(label "WIRE_B_IN"
 		(at 185.42 53.34 0)
 		(effects
@@
 		)
 	)
-	(label "WIRE_A_IN"
+	(label "THETA_A_IN"
 		(at 200.66 166.37 0)
 		(effects
@@
 		)
 	)
-	(label "THETA_A_IN"
+	(label "WIRE_A_IN"
 		(at 207.01 46.99 180)
 		(effects
@@
 			)
 		)
-		(property "Value" "THETA"
+		(property "Value" "WIRE"
 			(at 181.61 24.13 90)
 			(show_name no)
@@
 			)
 		)
-		(property "Value" "WIRE"
+		(property "Value" "THETA"
 			(at 196.85 130.8101 90)
 			(show_name no)
